File: PCB/Pynq Adapterboard.kicad_pcb (KiCad board)
At the start: 2 copper layers, 15 parts, among them J1 Conn_01x06_Pin

Commit message: pcb done
Parts:
- removed Motordrive1_PWR1: Conn_01x03_Pin, Connector_PinHeader_2.54mm:PinHeader_1x03_P2.54mm_Vertical
- PMODA1, PMODB1: footprint Connector_PinHeader_2.54mm:PinHeader_2x06_P2.54mm_Vertical -> Library:PinHeader_2x06_CORRECTED
- moved ultrasoon_1 130.7 mm to (52.7, 106.7), turned to 90 degrees
- moved Speedsensor_4 114.0 mm to (54.6, 138.1), turned to 90 degrees
- moved Speedsensor_3 111.4 mm to (50.8, 135.5), turned to 180 degrees
- moved ultrasoon_2 110.8 mm to (64.1, 106.7), turned to 90 degrees
- moved Motordrive2 104.5 mm to (59.7, 131.7), turned to 90 degrees
- moved PMODB1 87.1 mm to (60.9, 56.8), turned to 180 degrees
- moved PMODA1 86.6 mm to (54.6, 126.6), turned to 180 degrees
- moved Motordrive2_PWR1 81.4 mm to (67.3, 115.2)
- moved MPU6050 79.6 mm to (48.3, 67.3), turned to 90 degrees
- moved U1 78.5 mm to (68.6, 79.6), turned to -90 degrees
- moved J1 73.8 mm to (53.3, 73.7)
- moved Motordrive1 69.4 mm to (64.7, 37.7), turned to -90 degrees
- moved Speedsensor_2 52.9 mm to (49.5, 59.7), turned to 90 degrees
- moved Speedsensor_1 47.1 mm to (49.5, 55.9), turned to 90 degrees
Connections:
- Motordrive1 pad 4: Motor_Backwards_1 -> Motor_Forward_1
- Motordrive1 pad 5: Motor_Forward_1 -> Motor_Backwards_1
- Motordrive2 pad 4: Motor_Backward_3 -> Motor_Forward_3
- Motordrive2 pad 5: Motor_Forward_3 -> Motor_Backward_3
- U1 pad GND: GND -> (no net)
Routing:
- net Motor_Enable_1: track 0.00 -> 162.4 mm
- net +3.3V: track 0.00 -> 108.4 mm
- net Motor_Backward_3: track 0.00 -> 45.9 mm
- net Motor_Forward_3: track 0.00 -> 37.5 mm
- net +5V: track 27.1 -> 49.9 mm
- net Motor_Backwards_2: track 0.00 -> 19.9 mm
- net Motor_Forward_4: track 0.00 -> 18.1 mm
- net Motor_Forwards_2: track 0.00 -> 16.6 mm
- net Motor_Backwards_1: track 0.00 -> 16.3 mm
- net Motor_Backwards_4: track 0.00 -> 14.9 mm
- net GND: track 0.00 -> 14.3 mm
- net Motor_Forward_1: track 0.00 -> 13.7 mm
- net Speed_4: track 0.00 -> 13.5 mm
- net Speed_2: track 0.00 -> 8.85 mm
- net SDA: track 0.00 -> 6.35 mm
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- added copper zone on B.Cu, net GND
Other:
- board outline added: 31.7 x 111.8 mm
- board text added: "Seppe B. Kobe D."
