File: PCB/Pynq Adapterboard.kicad_sch (KiCad schematic)
At the start: 13 parts, among them J1 Conn_01x06_Pin

Commit message: pcb needs design
Parts:
- added MPU6050: Conn_01x08_Pin, Connector_PinHeader_2.54mm:PinHeader_1x08_P2.54mm_Vertical, symbol Connector:Conn_01x08_Pin
- added U1: ~, Library:KY-051, symbol New_Library:KY-051
- J1, Motordrive1, Motordrive2: footprint (none) -> Connector_PinHeader_2.54mm:PinHeader_1x06_P2.54mm_Vertical
- Motordrive1_PWR1: renamed from Motordrive1_PWR; footprint (none) -> Connector_PinHeader_2.54mm:PinHeader_1x03_P2.54mm_Vertical
- Motordrive2_PWR1: renamed from Motordrive2_PWR; footprint (none) -> Connector_PinHeader_2.54mm:PinHeader_1x03_P2.54mm_Vertical
- PMODA1: renamed from PMODA; footprint (none) -> Connector_PinHeader_2.54mm:PinHeader_2x06_P2.54mm_Vertical
- PMODB1: renamed from PMODB; footprint (none) -> Connector_PinHeader_2.54mm:PinHeader_2x06_P2.54mm_Vertical
- Speedsensor_1, Speedsensor_2, Speedsensor_3, Speedsensor_4: footprint (none) -> Connector_PinHeader_2.54mm:PinHeader_1x03_P2.54mm_Vertical
- ultrasoon_1, ultrasoon_2: footprint (none) -> Connector_PinHeader_2.54mm:PinHeader_1x04_P2.54mm_Vertical
Connections:
- net +3.3V: now also Speedsensor_1.1 (Pin_1), Speedsensor_2.1 (Pin_1), Speedsensor_3.1 (Pin_1), Speedsensor_4.1 (Pin_1), MPU6050.1 (Pin_1), U1. (VCCb)
- net +5V: now also U1. (VCCb)
- net GND: now also Speedsensor_1.2 (Pin_2), Speedsensor_2.2 (Pin_2), Speedsensor_3.2 (Pin_2), Speedsensor_4.2 (Pin_2), MPU6050.2 (Pin_2), U1. (VCCb)
- net Motor_Backwards_1: now also PMODB1.9 (Pin_9)
- net Motor_Forwards_2: now also PMODB1.4 (Pin_4)
- net Speed_4: now reaches PMODA1.1 (Pin_1)
- net Speed_4: now also Speedsensor_4.3 (Pin_3)
- net Motor_Forward_3: now reaches PMODA1.10 (Pin_10)
- net Motor_Forward_3: now also Motordrive2.5 (Pin_5)
- net Motor_Backwards_4: now reaches PMODA1.3 (Pin_3)
- net Motor_Backwards_4: now also Motordrive2.2 (Pin_2)
- net Motor_Forward_4: now reaches PMODA1.4 (Pin_4)
- net Motor_Forward_4: now also Motordrive2.3 (Pin_3)
- net Speed_3: now reaches PMODA1.7 (Pin_7)
- net Speed_3: now also Speedsensor_3.3 (Pin_3)
- net Motor_Backward_3: now reaches PMODA1.9 (Pin_9)
- net Motor_Backward_3: now also Motordrive2.4 (Pin_4)
- net SCL: now reaches J1.1 (Pin_1)
- net SCL: now also MPU6050.3 (Pin_3)
- net SDA: now reaches J1.2 (Pin_2)
- net SDA: now also MPU6050.4 (Pin_4)
- net ECHO_0_3.3V: now reaches J1.3 (Pin_3)
- net ECHO_0_3.3V: now also U1. (VCCb)
- net TRIGGER_0_3.3V: now reaches J1.4 (Pin_4)
- net TRIGGER_0_3.3V: now also U1. (VCCb)
- net ECHO_1_3.3V: now reaches J1.5 (Pin_5)
- net ECHO_1_3.3V: now also U1. (VCCb)
- net TRIGGER_1_3.3V: now reaches J1.6 (Pin_6)
- net TRIGGER_1_3.3V: now also U1. (VCCb)
- net Speed_2: now reaches PMODB1.1 (Pin_1)
- net Speed_2: now also Speedsensor_2.3 (Pin_3)
- net Motor_Backwards_2: now reaches PMODB1.3 (Pin_3)
- net Motor_Backwards_2: now also Motordrive1.2 (Pin_2)
- net Speed_1: now reaches PMODB1.7 (Pin_7)
- net Speed_1: now also Speedsensor_1.3 (Pin_3)
- net Motor_Enable_1: now reaches PMODB1.8 (Pin_8)
- net Motor_Enable_1: now also Motordrive1.1 (Pin_1), Motordrive1.6 (Pin_6), Motordrive2.1 (Pin_1), Motordrive2.6 (Pin_6)
- net ECHO_1_5V: now reaches ultrasoon_2.2 (Pin_2)
- net ECHO_1_5V: now also U1. (VCCb)
- net TRIGGER_1_5V: now reaches ultrasoon_2.3 (Pin_3)
- net TRIGGER_1_5V: now also U1. (VCCb)
- net ECHO_0_5V: now reaches ultrasoon_1.2 (Pin_2)
- net ECHO_0_5V: now also U1. (VCCb)
- net TRIGGER_0_5V: now reaches ultrasoon_1.3 (Pin_3)
- net TRIGGER_0_5V: now also U1. (VCCb)
Other:
- moved on the sheet: J1, Motordrive1, Motordrive1_PWR1, Motordrive2, Motordrive2_PWR1, PMODA1, PMODB1, Speedsensor_1, Speedsensor_2, Speedsensor_3, Speedsensor_4, ultrasoon_1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

Commit message: pcb done
Parts:
- PMODA1, PMODB1: footprint Connector_PinHeader_2.54mm:PinHeader_2x06_P2.54mm_Vertical -> Library:PinHeader_2x06_CORRECTED
Changed lines of the file:
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@@
       (effects (font (size 1.27 1.27)))
     )
-    (property "Footprint" "Connector_PinHeader_2.54mm:PinHeader_2x06_P2.54mm_Vertical" (at 46.99 50.8 0)
+    (property "Footprint" "Library:PinHeader_2x06_CORRECTED" (at 46.99 50.8 0)
       (effects (font (size 1.27 1.27)) hide)
     )
@@
       (effects (font (size 1.27 1.27)))
     )
-    (property "Footprint" "Connector_PinHeader_2.54mm:PinHeader_2x06_P2.54mm_Vertical" (at 46.99 76.2 0)
+    (property "Footprint" "Library:PinHeader_2x06_CORRECTED" (at 46.99 76.2 0)
       (effects (font (size 1.27 1.27)) hide)
     )
